File: EyeSPI-Featherwing.kicad_sch (KiCad schematic)
At the start: 24 parts, among them J101 Conn_01x16, J102 Conn_01x12, J103 Conn_01x07, J104 Conn_01x13, J105 Conn_01x06, J106 EYE_SPI_DISPLAY_FLIP, J107 Conn_01x01, J108 Conn_01x01, J109 Conn_01x01

Commit message: Closed #1
Parts:
- J106: value EYE_SPI_DISPLAY_FLIP -> EYE_SPI_DISPLAY_TYPE_B; symbol Resterampe:EYE_SPI_DISPLAY_FLIP -> Resterampe:EYE_SPI_DISPLAY_TYPE_B
Connections:
- net +3V3: now also J106.18 (VCC); no longer J106.1 (VCC)
- net BUSY: now also J106.3 (BUSY/TE); no longer J106.16 (BUSY/TE)
- net EYESPI_MISO: now also J106.13 (MISO); no longer J106.6 (MISO)
- net EYESPI_MOSI: now also J106.14 (MOSI); no longer J106.5 (MOSI)
- net EYESPI_SCK: now also J106.15 (SCK); no longer J106.4 (SCK)
- net EYESPI_SCL: now also J106.6 (SCL); no longer J106.13 (SCL)
- net EYESPI_SDA: now also J106.5 (SDA); no longer J106.14 (SDA)
- net GND: now also J106.16 (GND); no longer J106.3 (GND)
- net GPIO1: now also J106.2 (GPIO1); no longer J106.17 (GPIO1)
- net GPIO2: now also J106.1 (GPIO2); no longer J106.18 (GPIO2)
- net INT: now also J106.4 (INT); no longer J106.15 (INT)
- net LITE: now also J106.17 (BL); no longer J106.2 (BL)
- net TFT_DC: now also J106.12 (DC); no longer J106.7 (DC)
- net ~{CARD_CS}: now also J106.9 (~{SD_CS}); no longer J106.10 (~{SD_CS})
- net ~{MEM_CS}: now also J106.8 (~{MEM_CS}); no longer J106.11 (~{MEM_CS})
- net ~{TFT_CS}: now also J106.10 (~{DISP_CS}); no longer J106.9 (~{DISP_CS})
- net ~{TFT_RST}: now also J106.11 (~{RESET}); no longer J106.8 (~{RESET})
- net ~{TS_CS}: now also J106.7 (~{TS_CS}); no longer J106.12 (~{TS_CS})
Changed lines of the file:
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@@
   (title_block
     (title "EYESPI Feather Wing")
-    (date "2023-01-01")
-    (rev "1.0")
+    (date "2023-02-08")
+    (rev "2.0.0")
     (company "Resterampe Berlin")
     (comment 3 "https://creativecommons.org/licenses/by-nc/4.0")
@@
     (effects (font (size 1.27 1.27)) (justify left bottom))
   )
-  (symbol (lib_id "Resterampe:EYE_SPI_DISPLAY_FLIP") (at 67.31 140.97 0) (unit 1)
+  (symbol (lib_id "Resterampe:EYE_SPI_DISPLAY_TYPE_B") (at 67.31 140.97 0) (unit 1)
     (in_bom yes) (on_board yes)
     (property "Reference" "J106" (id 0) (at 69.85 170.18 0)
       (effects (font (size 1.9304 1.6408)) (justify left bottom))
     )
-    (property "Value" "EYE_SPI_DISPLAY_FLIP" (id 1) (at 74.93 154.94 90)
+    (property "Value" "EYE_SPI_DISPLAY_TYPE_B" (id 1) (at 74.93 154.94 90)
       (effects (font (size 1.9304 1.6408)) (justify left bottom))
     )
-    (property "Footprint" "Connector_FFC-FPC:Hirose_FH12-18S-0.5SH_1x18-1MP_P0.50mm_Horizontal" (id 2) (at 67.31 140.97 0)
-      (effects (font (size 1.27 1.27)) hide)
-    )
-    (property "Datasheet" "https://learn.adafruit.com/adafruit-eyespi-breakout-board/pinouts" (id 3) (at 67.31 140.97 0)
+    (property "Footprint" "Connector_FFC-FPC:Hirose_FH12-18S-0.5SH_1x18-1MP_P0.50mm_Horizontal" (id 2) (at 67.31 187.96 0)
+      (effects (font (size 1.27 1.27)) hide)
+    )
+    (property "Datasheet" "https://learn.adafruit.com/adafruit-eyespi-breakout-board/pinouts" (id 3) (at 66.04 191.77 0)
       (effects (font (size 1.27 1.27)) hide)
     )
@@
     )
     (path "/08eeb292-5bb1-4093-89ce-08ec8a892adb"
-      (reference "J106") (unit 1) (value "EYE_SPI_DISPLAY_FLIP") (footprint "Connector_FFC-FPC:Hirose_FH12-18S-0.5SH_1x18-1MP_P0.50mm_Horizontal")
+      (reference "J106") (unit 1) (value "EYE_SPI_DISPLAY_TYPE_B") (footprint "Connector_FFC-FPC:Hirose_FH12-18S-0.5SH_1x18-1MP_P0.50mm_Horizontal")
     )
     (path "/b94809a9-ed99-4dad-a433-ca0fc388ba07"
