File: EyeSPI-Featherwing.kicad_pcb (KiCad board)
At the start: 4 copper layers, 50.8 x 22.9 mm, 34 parts, among them J101 Conn_01x16, J102 Conn_01x12, J106 EYE_SPI_DISPLAY_FLIP, J107 Conn_01x01, J108 Conn_01x01, J109 Conn_01x01

Commit message: Closed #1
Parts:
- J106: value EYE_SPI_DISPLAY_FLIP -> EYE_SPI_DISPLAY_TYPE_B
- moved J109 12.5 mm to (143.8, 98.3)
- moved J107 12.2 mm to (140.6, 98.3)
- moved J108 12.0 mm to (137.3, 98.3)
- moved kibuzzard-63C5DD9E 11.7 mm to (140.4, 101.4), turned to 90 degrees
- moved kibuzzard-63C5DDB7 11.5 mm to (143.8, 102.7), turned to 90 degrees
- moved kibuzzard-63C5DDAE 11.4 mm to (137.3, 101.5), turned to 90 degrees
Connections:
- J106 pad 1: +3V3 -> /GPIO2
- J106 pad 10: /~{CARD_CS} -> /~{TFT_CS}
- J106 pad 11: /~{MEM_CS} -> /~{TFT_RST}
- J106 pad 12: /~{TS_CS} -> /TFT_DC
- J106 pad 13: /EYESPI_SCL -> /EYESPI_MISO
- J106 pad 14: /EYESPI_SDA -> /EYESPI_MOSI
- J106 pad 15: /INT -> /EYESPI_SCK
- J106 pad 16: /BUSY -> GND
- J106 pad 17: /GPIO1 -> /LITE
- J106 pad 18: /GPIO2 -> +3V3
- J106 pad 2: /LITE -> /GPIO1
- J106 pad 3: GND -> /BUSY
- J106 pad 4: /EYESPI_SCK -> /INT
- J106 pad 5: /EYESPI_MOSI -> /EYESPI_SDA
- J106 pad 6: /EYESPI_MISO -> /EYESPI_SCL
- J106 pad 7: /TFT_DC -> /~{TS_CS}
- J106 pad 8: /~{TFT_RST} -> /~{MEM_CS}
- J106 pad 9: /~{TFT_CS} -> /~{CARD_CS}
Routing:
- net +3V3: track 13.6 -> 30.3 mm, vias 1 -> 0
- net /LITE: track 18.5 -> 4.44 mm
- net /EYESPI_MISO: track 37.9 -> 28.2 mm, vias 2 -> 0
- net /EYESPI_SCK: track 31.9 -> 22.8 mm, vias 2 -> 0
- net /EYESPI_MOSI: track 34.6 -> 25.5 mm, vias 2 -> 0
- net /BUSY: track 20.2 -> 14.4 mm
- net /~{TFT_RST}: track 28.7 -> 34.2 mm
- net /INT: track 21.9 -> 17.1 mm, vias 2 -> 0
- net /TFT_DC: track 26.2 -> 30.6 mm
- net /GPIO1: track 12.8 -> 8.57 mm
- net /~{MEM_CS}: track 21.5 -> 18.2 mm
- net /GPIO2: track 8.14 -> 5.13 mm
- net /EYESPI_SDA: track 38.8 -> 36.4 mm, vias 2 -> 0
- net GND: track 3.56 -> 1.58 mm, vias 2 -> 12
- net unconnected-(J106-PadMP): track 14.2 -> 12.3 mm
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- added copper zone on F.Cu, net GND
- removed copper zone on F.Cu, net +3V3
Other:
- copper layers 4 -> 2
- board text removed: "CHECK FOOTPRINT!"

Commit message: Production
Parts:
- added kibuzzard-63E91F4E: G***, kibuzzard-63E91F4E, F.Cu at (125.4, 105.0)
Routing:
- net GND: vias 12 -> 11
